Commit message: modified

File: arm_car_rviz_simulation/urdf/ur10_car.urdf.xacro (robot description, xacro)
@@ -21,5 +21,5 @@
     <parent link="head" />
     <child link = "ur_base_link" />
-    <origin xyz="0.0 0.0 0.0" rpy="0.0 0.0 0.0" />
+    <origin xyz="0.0 0.0 0.0" rpy="0.0 0.0 3.1415926" />
   </joint>
 </robot>
